File: agat_disk_adapter.kicad_sch (KiCad schematic)
At the start: 14 parts, among them J1 IDC‐20, J2 IDC‐20, J3 IDC‐34, J4 IDC‐10, J5 KK‐4

Commit message: made "fan" conn pads 2.18 - close to library's 2.19, and aligned to 0.01 grid; fixed title info
Other:
- company: Михаил Шевченко mike.shevchenko@gmail.com КИБЕР-МУЗЕЙ, МУРОМ -> КИБЕР-МУЗЕЙ, МУРОМ - Михаил Шевченко - mike.shevchenko@gmail.com
Changed lines of the file:
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@@
 		(date "2026-09")
 		(rev "V1")
-		(company "Михаил Шевченко mike.shevchenko@gmail.com КИБЕР-МУЗЕЙ, МУРОМ")
+		(company "КИБЕР-МУЗЕЙ, МУРОМ - Михаил Шевченко - mike.shevchenko@gmail.com")
 		(comment 1 "- Подключение КНГМД - штатным кабелем, либо шлейфом с СНП34-30 на IDC-20,")
 		(comment 2 "- Сигнал \"Выбор Блока\" для 2-го дисковода (ВБ2) можно завести через -12|DE2.")
